Commit message: added main file for test teleop-retarget, also added assets

File: assets/aiw/ffw_bh5_rev1_follower/ffw_bh5_follower_alone.urdf (robot description, URDF)
Before this commit: robot ffw_bh5_follower, 81 links, 80 joints
Links:
- link camera_l_link: geometry collision box size=0.023 0.042 0.042; visual mesh filename=../rs_meshes/d405.stl scale=0.001 0.001 0.001
- link camera_r_link: geometry collision box size=0.023 0.042 0.042; visual mesh filename=../rs_meshes/d405.stl scale=0.001 0.001 0.001
- link zedm_camera_center: geometry collision mesh filename=../rs_meshes/d405.stl scale=0.001 0.001 0.001; visual mesh filename=../rs_meshes/d405.stl scale=0.001 0.001 0.001
